File: hardware/wavelength keyboard v0.0.kicad_sch (KiCad schematic)
At the start: 1 part, among them U1 nRF52840

Commit message: session #3 content
Parts:
- added C1: 1.5pF, Capacitor_SMD:C_0402_1005Metric, symbol Device:C
- added C2, C5: 1pF, Capacitor_SMD:C_0402_1005Metric, symbol Device:C
- added C3, C4: 12pF, Capacitor_SMD:C_0402_1005Metric, symbol Device:C
- added L1: 4.7nH, Inductor_SMD:L_0402_1005Metric, symbol Device:L
- added R1: 50, Resistor_SMD:R_0402_1005Metric, symbol Device:R
- added Y1: 32MHz, Crystal:Crystal_SMD_2016-4Pin_2.0x1.6mm, symbol Device:Crystal
Connections:
- net GND: now also C1.2, C2.2, C3.2, C4.2
- net VSS_ANT: now also C5.2
- net at U1.A23 (XC2): now also C4.1, Y1.2
- net at U1.B24 (XC1): now also C3.1, Y1.1
- net at U1.H23 (ANT): now also C5.1, L1.2
- new net: C2.1, L1.1, R1.1
- new net Antenna: C1.1, R1.2
Other:
- moved on the sheet: U1
